File: hardware/dsp_som/dsp_som.kicad_pcb (KiCad board)
At the start: 2 copper layers, 40 x 60 mm, 12 parts, among them J1 Micro_SD_Card_Det_Hirose_DM3AT, J2 Conn_02x07_Odd_Even, J3 Conn_02x22_Odd_Even, U1 IS42S16400J-xT, U2 SGTL5000XNAA3, U4 BU18SD2MG-MTR, U5 STM32F446ZCTx, Y1 16MHz, Y3 32kHz768

Commit message: 1st attempt at routing the SDRAM
Parts:
- added C10: 100n, Capacitor_SMD:C_0402_1005Metric, B.Cu at (98.0, 75.1)
- added C11: 100n, Capacitor_SMD:C_0402_1005Metric, B.Cu at (99.0, 86.5)
- added C12: 100n, Capacitor_SMD:C_0402_1005Metric, B.Cu at (106.0, 88.1)
- added C13: 100n, Capacitor_SMD:C_0402_1005Metric, B.Cu at (111.0, 88.0)
- added C14: 100n, Capacitor_SMD:C_0402_1005Metric, B.Cu at (117.9, 86.3)
- added C15: 100n, Capacitor_SMD:C_0402_1005Metric, B.Cu at (122.0, 70.8)
- added C16: 1u, Capacitor_SMD:C_0603_1608Metric, B.Cu at (122.0, 69.5)
- added C17: 4.7u, Capacitor_SMD:C_0603_1608Metric, B.Cu at (116.3, 85.8)
- added C18: 10p, Capacitor_SMD:C_0402_1005Metric, F.Cu at (126.5, 71.0)
- added C19: 10p, Capacitor_SMD:C_0402_1005Metric, F.Cu at (126.5, 77.0)
- added C2: 100n, Capacitor_SMD:C_0402_1005Metric, B.Cu at (122.0, 74.8)
- added C20: ??, Capacitor_SMD:C_0402_1005Metric, F.Cu at (125.5, 86.0)
- added C21: ??, Capacitor_SMD:C_0402_1005Metric, F.Cu at (125.5, 83.0)
- added C22: 100n, Capacitor_SMD:C_0402_1005Metric, B.Cu at (98.6, 61.6)
- added C23: 100n, Capacitor_SMD:C_0402_1005Metric, B.Cu at (101.4, 62.7)
- added C24: 100n, Capacitor_SMD:C_0402_1005Metric, B.Cu at (103.8, 62.7)
- added C25: 100n, Capacitor_SMD:C_0402_1005Metric, B.Cu at (108.2, 62.1)
- added C26: 100n, Capacitor_SMD:C_0402_1005Metric, B.Cu at (119.4, 61.5)
- added C27: 100n, Capacitor_SMD:C_0402_1005Metric, B.Cu at (101.4, 51.2)
- added C28: 100n, Capacitor_SMD:C_0402_1005Metric, B.Cu at (106.2, 51.2)
- added C29: 100n, Capacitor_SMD:C_0402_1005Metric, B.Cu at (122.0, 72.2)
- added C3: 100n, Capacitor_SMD:C_0402_1005Metric, B.Cu at (118.0, 83.7)
- added C30: 1u, Capacitor_SMD:C_0603_1608Metric, B.Cu at (122.0, 73.5)
- added C31: 100n, Capacitor_SMD:C_0402_1005Metric, B.Cu at (99.0, 80.0)
- added C32: 1u, Capacitor_SMD:C_0603_1608Metric, B.Cu at (100.3, 80.0)
- added C33: 1u, Capacitor_SMD:C_0603_1608Metric, F.Cu at (103.2, 92.5)
- added C34: 1u, Capacitor_SMD:C_0603_1608Metric, F.Cu at (103.2, 95.0)
- added C4: 100n, Capacitor_SMD:C_0402_1005Metric, B.Cu at (119.0, 79.0)
- added C5: 100n, Capacitor_SMD:C_0402_1005Metric, B.Cu at (119.0, 71.5)
- added C6: 100n, Capacitor_SMD:C_0402_1005Metric, B.Cu at (117.0, 68.0)
- added C7: 100n, Capacitor_SMD:C_0402_1005Metric, B.Cu at (110.5, 68.0)
- added C8: 100n, Capacitor_SMD:C_0402_1005Metric, B.Cu at (105.5, 68.0)
- added C9: 100n, Capacitor_SMD:C_0402_1005Metric, B.Cu at (99.8, 68.0)
- added R1: 10R, Resistor_SMD:R_0402_1005Metric, F.Cu at (122.1, 75.2)
- added R2: 100k, Resistor_SMD:R_0402_1005Metric, F.Cu at (114.0, 92.0)
- J2: value Conn_02x07_Odd_Even -> SWD
- moved Y3 19.1 mm to (123.0, 84.0), turned to 90 degrees
- moved J2 16.0 mm to (125.0, 64.0)
- moved Y1 3.16 mm to (126.0, 74.0), turned to 0 degrees
- moved U5 1.00 mm to (109.0, 78.0), turned to 180 degrees
Connections:
- J2 pad 11: unconnected-(J2-Pin_11-Pad11) -> GND
- J2 pad 12: unconnected-(J2-Pin_12-Pad12) -> /nRST
- J2 pad 13: unconnected-(J2-Pin_13-Pad13) -> /VCP_RX
- J2 pad 14: unconnected-(J2-Pin_14-Pad14) -> /VCP_TX
- J2 pad 3: unconnected-(J2-Pin_3-Pad3) -> +3.3V
- J2 pad 4: unconnected-(J2-Pin_4-Pad4) -> /SWDIO
- J2 pad 5: unconnected-(J2-Pin_5-Pad5) -> GND
- J2 pad 6: unconnected-(J2-Pin_6-Pad6) -> /SWCLK
- J2 pad 7: unconnected-(J2-Pin_7-Pad7) -> GND
- J2 pad 8: unconnected-(J2-Pin_8-Pad8) -> /SWO
- U1 pad 1: Net-(U1-VDD-Pad1) -> +3.3V
- U1 pad 10: unconnected-(U1-DQ5-Pad10) -> /DQ5
- U1 pad 11: unconnected-(U1-DQ6-Pad11) -> /DQ6
- U1 pad 12: Net-(U1-GNDQ-Pad12) -> GND
- U1 pad 13: unconnected-(U1-DQ7-Pad13) -> /DQ7
- U1 pad 14: Net-(U1-VDD-Pad1) -> +3.3V
- U1 pad 15: unconnected-(U1-LDQM-Pad15) -> /LDQM
- U1 pad 16: unconnected-(U1-~{WE}-Pad16) -> /nWE
- U1 pad 17: unconnected-(U1-~{CAS}-Pad17) -> /nCAS
- U1 pad 18: unconnected-(U1-~{RAS}-Pad18) -> /nRAS
- U1 pad 19: unconnected-(U1-~{CS}-Pad19) -> /nCS
- U1 pad 2: unconnected-(U1-DQ0-Pad2) -> /DQ0
- U1 pad 20: unconnected-(U1-BA0-Pad20) -> /BA0
- U1 pad 21: unconnected-(U1-BA1-Pad21) -> /BA1
- U1 pad 22: unconnected-(U1-A10-Pad22) -> /A10
- U1 pad 23: unconnected-(U1-A0-Pad23) -> /A0
- U1 pad 24: unconnected-(U1-A1-Pad24) -> /A1
- U1 pad 25: unconnected-(U1-A2-Pad25) -> /A2
- U1 pad 26: unconnected-(U1-A3-Pad26) -> /A3
- U1 pad 27: Net-(U1-VDD-Pad1) -> +3.3V
- U1 pad 28: Net-(U1-GND-Pad28) -> GND
- U1 pad 29: unconnected-(U1-A4-Pad29) -> /A4
- U1 pad 3: Net-(U1-VDDQ-Pad3) -> +3.3V
- U1 pad 30: unconnected-(U1-A5-Pad30) -> /A5
- U1 pad 31: unconnected-(U1-A6-Pad31) -> /A6
- U1 pad 32: unconnected-(U1-A7-Pad32) -> /A7
- U1 pad 33: unconnected-(U1-A8-Pad33) -> /A8
- U1 pad 34: unconnected-(U1-A9-Pad34) -> /A9
- U1 pad 35: unconnected-(U1-A11-Pad35) -> /A11
- U1 pad 37: unconnected-(U1-CKE-Pad37) -> /CKE
- U1 pad 38: unconnected-(U1-CLK-Pad38) -> /CLK
- U1 pad 39: unconnected-(U1-UDQM-Pad39) -> /UDQM
- U1 pad 4: unconnected-(U1-DQ1-Pad4) -> /DQ1
- U1 pad 41: Net-(U1-GND-Pad28) -> GND
- U1 pad 42: unconnected-(U1-DQ8-Pad42) -> /DQ8
- U1 pad 43: Net-(U1-VDDQ-Pad3) -> +3.3V
- U1 pad 44: unconnected-(U1-DQ9-Pad44) -> /DQ9
- U1 pad 45: unconnected-(U1-DQ10-Pad45) -> /DQ10
- U1 pad 46: Net-(U1-GNDQ-Pad12) -> GND
- U1 pad 47: unconnected-(U1-DQ11-Pad47) -> /DQ11
- U1 pad 48: unconnected-(U1-DQ12-Pad48) -> /DQ12
- U1 pad 49: Net-(U1-VDDQ-Pad3) -> +3.3V
- U1 pad 5: unconnected-(U1-DQ2-Pad5) -> /DQ2
- U1 pad 50: unconnected-(U1-DQ13-Pad50) -> /DQ13
- U1 pad 51: unconnected-(U1-DQ14-Pad51) -> /DQ14
- U1 pad 52: Net-(U1-GNDQ-Pad12) -> GND
- U1 pad 53: unconnected-(U1-DQ15-Pad53) -> /DQ15
- U1 pad 54: Net-(U1-GND-Pad28) -> GND
- U1 pad 6: Net-(U1-GNDQ-Pad12) -> GND
- U1 pad 7: unconnected-(U1-DQ3-Pad7) -> /DQ3
- U1 pad 8: unconnected-(U1-DQ4-Pad8) -> /DQ4
- U1 pad 9: Net-(U1-VDDQ-Pad3) -> +3.3V
- U2 pad 1: Net-(U2-GND-Pad1) -> GND
- U2 pad 3: Net-(U2-GND-Pad1) -> GND
- U2 pad 33: Net-(U2-GND-Pad1) -> GND
- U2 pad 7: unconnected-(U2-AGND-Pad7) -> GND
- U4 pad 1: unconnected-(U4-IN-Pad1) -> +3.3V
- U4 pad 2: unconnected-(U4-GND-Pad2) -> GND
- U4 pad 3: unconnected-(U4-STBY-Pad3) -> +3.3V
- U4 pad 5: unconnected-(U4-OUT-Pad5) -> +1V8
- U5 pad 10: unconnected-(U5-PF0-Pad10) -> /A0
- U5 pad 105: unconnected-(U5-PA13-Pad105) -> /SWDIO
- U5 pad 107: Net-(U5-VSS-Pad107) -> GND
- U5 pad 108: unconnected-(U5-VDD-Pad108) -> +3.3V
- U5 pad 109: unconnected-(U5-PA14-Pad109) -> /SWCLK
- U5 pad 11: unconnected-(U5-PF1-Pad11) -> /A1
- U5 pad 114: unconnected-(U5-PD0-Pad114) -> /DQ2
- U5 pad 115: unconnected-(U5-PD1-Pad115) -> /DQ3
- U5 pad 12: unconnected-(U5-PF2-Pad12) -> /A2
- U5 pad 120: Net-(U5-VSS-Pad107) -> GND
- U5 pad 121: unconnected-(U5-VDD-Pad121) -> +3.3V
- U5 pad 13: unconnected-(U5-PF3-Pad13) -> /A3
- U5 pad 130: Net-(U5-VSS-Pad107) -> GND
- U5 pad 131: unconnected-(U5-VDD-Pad131) -> +3.3V
- U5 pad 132: unconnected-(U5-PG15-Pad132) -> /nCAS
- U5 pad 133: unconnected-(U5-PB3-Pad133) -> /SWO
- U5 pad 135: unconnected-(U5-PB5-Pad135) -> /CKE
- U5 pad 136: unconnected-(U5-PB6-Pad136) -> /nCS
- U5 pad 138: unconnected-(U5-BOOT0-Pad138) -> /BOOT0
- U5 pad 14: unconnected-(U5-PF4-Pad14) -> /A4
- U5 pad 141: unconnected-(U5-PE0-Pad141) -> /LDQM
- U5 pad 142: unconnected-(U5-PE1-Pad142) -> /UDQM
- U5 pad 143: unconnected-(U5-PDR_ON-Pad143) -> +3.3V
- U5 pad 144: unconnected-(U5-VDD-Pad144) -> +3.3V
- U5 pad 15: unconnected-(U5-PF5-Pad15) -> /A5
- U5 pad 16: Net-(U5-VSS-Pad107) -> GND
- U5 pad 17: unconnected-(U5-VDD-Pad17) -> +3.3V
- U5 pad 23: unconnected-(U5-PH0-Pad23) -> /OSC_IN
- U5 pad 24: unconnected-(U5-PH1-Pad24) -> /OSC_OUT
- U5 pad 25: unconnected-(U5-NRST-Pad25) -> /nRST
- U5 pad 26: unconnected-(U5-PC0-Pad26) -> /nWE
- U5 pad 30: unconnected-(U5-VDD-Pad30) -> +3.3V
- U5 pad 31: unconnected-(U5-VSSA-Pad31) -> GND
- U5 pad 32: unconnected-(U5-VREF+-Pad32) -> +3.3V
- U5 pad 33: unconnected-(U5-VDDA-Pad33) -> +3.3VA
- U5 pad 38: Net-(U5-VSS-Pad107) -> GND
- U5 pad 39: unconnected-(U5-VDD-Pad39) -> +3.3V
- U5 pad 49: unconnected-(U5-PF11-Pad49) -> /nRAS
- U5 pad 50: unconnected-(U5-PF12-Pad50) -> /A6
- U5 pad 51: Net-(U5-VSS-Pad107) -> GND
- U5 pad 52: unconnected-(U5-VDD-Pad52) -> +3.3V
- U5 pad 53: unconnected-(U5-PF13-Pad53) -> /A7
- U5 pad 54: unconnected-(U5-PF14-Pad54) -> /A8
- U5 pad 55: unconnected-(U5-PF15-Pad55) -> /A9
- U5 pad 56: unconnected-(U5-PG0-Pad56) -> /A10
- U5 pad 57: unconnected-(U5-PG1-Pad57) -> /A11
- U5 pad 58: unconnected-(U5-PE7-Pad58) -> /DQ4
- U5 pad 59: unconnected-(U5-PE8-Pad59) -> /DQ5
- U5 pad 6: unconnected-(U5-VBAT-Pad6) -> +3.3V
- U5 pad 60: unconnected-(U5-PE9-Pad60) -> /DQ6
- U5 pad 61: Net-(U5-VSS-Pad107) -> GND
- U5 pad 62: unconnected-(U5-VDD-Pad62) -> +3.3V
- U5 pad 63: unconnected-(U5-PE10-Pad63) -> /DQ7
- U5 pad 64: unconnected-(U5-PE11-Pad64) -> /DQ8
- U5 pad 65: unconnected-(U5-PE12-Pad65) -> /DQ9
- U5 pad 66: unconnected-(U5-PE13-Pad66) -> /DQ10
- U5 pad 67: unconnected-(U5-PE14-Pad67) -> /DQ11
- U5 pad 68: unconnected-(U5-PE15-Pad68) -> /DQ12
- U5 pad 72: unconnected-(U5-VDD-Pad72) -> +3.3V
- U5 pad 77: unconnected-(U5-PD8-Pad77) -> /DQ13
- U5 pad 78: unconnected-(U5-PD9-Pad78) -> /DQ14
- U5 pad 79: unconnected-(U5-PD10-Pad79) -> /DQ15
- U5 pad 8: unconnected-(U5-PC14-Pad8) -> /OSC32_IN
- U5 pad 83: Net-(U5-VSS-Pad107) -> GND
- U5 pad 84: unconnected-(U5-VDD-Pad84) -> +3.3V
- U5 pad 85: unconnected-(U5-PD14-Pad85) -> /DQ0
- U5 pad 86: unconnected-(U5-PD15-Pad86) -> /DQ1
- U5 pad 89: unconnected-(U5-PG4-Pad89) -> /BA0
- U5 pad 9: unconnected-(U5-PC15-Pad9) -> /OSC32_OUT
- U5 pad 90: unconnected-(U5-PG5-Pad90) -> /BA1
- U5 pad 93: unconnected-(U5-PG8-Pad93) -> /CLK
- U5 pad 94: Net-(U5-VSS-Pad107) -> GND
- U5 pad 95: unconnected-(U5-VDDUSB-Pad95) -> +3.3V
- Y1 pad 1: unconnected-(Y1-Pad1) -> /XTAL_OUT
- Y1 pad 2: unconnected-(Y1-Pad2) -> GND
- Y1 pad 3: unconnected-(Y1-Pad3) -> /OSC_IN
- Y1 pad 4: unconnected-(Y1-Pad4) -> GND
- Y3 pad 1: unconnected-(Y3-Pad1) -> /OSC32_OUT
- Y3 pad 2: unconnected-(Y3-Pad2) -> /OSC32_IN
Routing:
- net +3.3V: track 0.00 -> 42.3 mm, vias 0 -> 22
- net /CLK: track 0.00 -> 40.5 mm, vias 0 -> 2
- net GND: track 0.00 -> 39.8 mm, vias 0 -> 33
- net /UDQM: track 0.00 -> 39.3 mm, vias 0 -> 2
- net /CKE: track 0.00 -> 37.4 mm, vias 0 -> 2
- net /LDQM: track 0.00 -> 36.8 mm, vias 0 -> 2
- net /A11: track 0.00 -> 34.1 mm, vias 0 -> 2
- net /BA0: track 0.00 -> 33.9 mm, vias 0 -> 2
- net /BA1: track 0.00 -> 33.5 mm, vias 0 -> 2
- net /DQ3: track 0.00 -> 32.4 mm, vias 0 -> 2
- net /DQ2: track 0.00 -> 32.0 mm, vias 0 -> 2
- net /A4: track 0.00 -> 31.9 mm, vias 0 -> 2
- net /A9: track 0.00 -> 31.7 mm, vias 0 -> 2
- net /A5: track 0.00 -> 30.3 mm, vias 0 -> 2
- net /A8: track 0.00 -> 30.0 mm, vias 0 -> 2
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- added copper zone on In2.Cu, net +3.3V
- added copper zone on In1.Cu, net GND
- added copper zone on In4.Cu, net GND
Other:
- copper layers 2 -> 6
- board text added: "Hole to hole 0.5mm - Center to center 0.8mm Via to via same net 0.254mm"
- board text removed: "Hole to hole 0.5mm Via to via same net 0.254mm"

Commit message: routing 1st version
Parts:
- added C35: 100n, Capacitor_SMD:C_0402_1005Metric, B.Cu at (100.2, 107.5)
- added C36: 100n, Capacitor_SMD:C_0402_1005Metric, B.Cu at (98.5, 103.2)
- added C37: 100n, Capacitor_SMD:C_0402_1005Metric, B.Cu at (100.2, 102.5)
- added C38: 100n, Capacitor_SMD:C_0402_1005Metric, B.Cu at (103.5, 104.0)
- added C39: 2.2u, Capacitor_SMD:C_0603_1608Metric, B.Cu at (97.7, 86.0)
- added C40: 2.2u, Capacitor_SMD:C_0603_1608Metric, B.Cu at (99.3, 66.7)
- added R3: 47k, Resistor_SMD:R_0402_1005Metric, F.Cu at (101.7, 96.2)
- added R4: 47k, Resistor_SMD:R_0402_1005Metric, F.Cu at (103.2, 95.6)
- added R5: 47k, Resistor_SMD:R_0402_1005Metric, F.Cu at (111.3, 91.7)
- added R6: 47k, Resistor_SMD:R_0402_1005Metric, F.Cu at (106.6, 93.3)
- added R7: 47k, Resistor_SMD:R_0402_1005Metric, F.Cu at (105.1, 94.0)
- added R8: 1.5k, Resistor_SMD:R_0402_1005Metric, F.Cu at (109.7, 103.1)
- added R9: 1.5k, Resistor_SMD:R_0402_1005Metric, F.Cu at (109.7, 105.3)
- moved U4 8.90 mm to (106.0, 100.5), turned to -90 degrees
- moved C34 7.88 mm to (108.5, 100.8), turned to 90 degrees
- moved C18 7.25 mm to (125.6, 78.2)
- moved U2 6.40 mm to (101.0, 105.0), turned to -90 degrees
- moved C33 6.06 mm to (106.5, 97.6), turned to 180 degrees
- moved R2 4.51 mm to (118.5, 91.5), turned to 180 degrees
- moved C19 4.10 mm to (125.6, 73.0)
- moved C1 3.04 mm to (102.0, 100.8)
- moved C20 2.96 mm to (125.8, 83.0), turned to 90 degrees
- moved FB1 2.58 mm to (102.0, 99.2), turned to 180 degrees
- moved C2 2.26 mm to (119.7, 75.0), turned to 180 degrees
- moved Y3 2.19 mm to (123.9, 82.0)
- moved C21 2.07 mm to (125.8, 81.0), turned to -90 degrees
- moved Y1 1.65 mm to (125.6, 75.6), turned to -90 degrees
Connections:
- J1 pad 1: unconnected-(J1-DAT2-Pad1) -> /SD_DAT2
- J1 pad 10: unconnected-(J1-DET_A-Pad10) -> /SD_DETECT
- J1 pad 11: unconnected-(J1-SHIELD-Pad11) -> GND
- J1 pad 2: unconnected-(J1-DAT3/CD-Pad2) -> /SD_DAT3
- J1 pad 3: unconnected-(J1-CMD-Pad3) -> /SD_CMD
- J1 pad 4: unconnected-(J1-VDD-Pad4) -> +3.3V
- J1 pad 5: unconnected-(J1-CLK-Pad5) -> /SD_CLK
- J1 pad 6: unconnected-(J1-VSS-Pad6) -> GND
- J1 pad 7: unconnected-(J1-DAT0-Pad7) -> /SD_DAT0
- J1 pad 8: unconnected-(J1-DAT1-Pad8) -> /SD_DAT1
- J1 pad 9: unconnected-(J1-DET_B-Pad9) -> GND
- J3 pad 1: unconnected-(J3-Pin_1-Pad1) -> +3.3V
- J3 pad 10: unconnected-(J3-Pin_10-Pad10) -> GND
- J3 pad 11: unconnected-(J3-Pin_11-Pad11) -> /ADC3_IN2
- J3 pad 12: unconnected-(J3-Pin_12-Pad12) -> GND
- J3 pad 13: unconnected-(J3-Pin_13-Pad13) -> /ADC3_IN3
- J3 pad 14: unconnected-(J3-Pin_14-Pad14) -> GND
- J3 pad 15: unconnected-(J3-Pin_15-Pad15) -> /ADC3_IN13
- J3 pad 16: unconnected-(J3-Pin_16-Pad16) -> GND
- J3 pad 17: unconnected-(J3-Pin_17-Pad17) -> /ADC3_IN12
- J3 pad 18: unconnected-(J3-Pin_18-Pad18) -> GND
- J3 pad 19: unconnected-(J3-Pin_19-Pad19) -> /ADC3_IN11
- J3 pad 2: unconnected-(J3-Pin_2-Pad2) -> GND
- J3 pad 20: unconnected-(J3-Pin_20-Pad20) -> GND
- J3 pad 21: unconnected-(J3-Pin_21-Pad21) -> /ADC3_IN8
- J3 pad 22: unconnected-(J3-Pin_22-Pad22) -> GND
- J3 pad 23: unconnected-(J3-Pin_23-Pad23) -> /ADC3_IN7
- J3 pad 24: unconnected-(J3-Pin_24-Pad24) -> GND
- J3 pad 25: unconnected-(J3-Pin_25-Pad25) -> /USB_DM
- J3 pad 26: unconnected-(J3-Pin_26-Pad26) -> GND
- J3 pad 27: unconnected-(J3-Pin_27-Pad27) -> /USB_DP
- J3 pad 28: unconnected-(J3-Pin_28-Pad28) -> GND
- J3 pad 29: unconnected-(J3-Pin_29-Pad29) -> /ADC3_IN6
- J3 pad 3: unconnected-(J3-Pin_3-Pad3) -> /PB10
- J3 pad 30: unconnected-(J3-Pin_30-Pad30) -> GND
- J3 pad 31: unconnected-(J3-Pin_31-Pad31) -> /ADC3_IN5
- J3 pad 32: unconnected-(J3-Pin_32-Pad32) -> GND
- J3 pad 33: unconnected-(J3-Pin_33-Pad33) -> /ADC3_IN4
- J3 pad 34: unconnected-(J3-Pin_34-Pad34) -> GND
- J3 pad 35: unconnected-(J3-Pin_35-Pad35) -> GND
- J3 pad 36: unconnected-(J3-Pin_36-Pad36) -> GND
- J3 pad 37: unconnected-(J3-Pin_37-Pad37) -> /LINEOUT_R
- J3 pad 38: unconnected-(J3-Pin_38-Pad38) -> GND
- J3 pad 39: unconnected-(J3-Pin_39-Pad39) -> /LINEOUT_L
- J3 pad 4: unconnected-(J3-Pin_4-Pad4) -> GND
- J3 pad 40: unconnected-(J3-Pin_40-Pad40) -> GND
- J3 pad 41: unconnected-(J3-Pin_41-Pad41) -> /LINEIN_R
- J3 pad 42: unconnected-(J3-Pin_42-Pad42) -> GND
- J3 pad 43: unconnected-(J3-Pin_43-Pad43) -> /LINEIN_L
- J3 pad 44: unconnected-(J3-Pin_44-Pad44) -> GND
- J3 pad 5: unconnected-(J3-Pin_5-Pad5) -> /PB11
- J3 pad 6: unconnected-(J3-Pin_6-Pad6) -> GND
- J3 pad 7: unconnected-(J3-Pin_7-Pad7) -> /PD12
- J3 pad 8: unconnected-(J3-Pin_8-Pad8) -> GND
- J3 pad 9: unconnected-(J3-Pin_9-Pad9) -> /PD13
- U2 pad 10: unconnected-(U2-VAG-Pad10) -> /VAG
- U2 pad 11: unconnected-(U2-LINEOUT_R-Pad11) -> /LINEOUT_R
- U2 pad 12: unconnected-(U2-LINEOUT_L-Pad12) -> /LINEOUT_L
- U2 pad 13: unconnected-(U2-LINEIN_R-Pad13) -> /LINEIN_R
- U2 pad 14: unconnected-(U2-LINEIN_L-Pad14) -> /LINEIN_L
- U2 pad 20: unconnected-(U2-VDDIO-Pad20) -> +3.3V
- U2 pad 21: unconnected-(U2-SYS_MCLK-Pad21) -> /CODEC_MCLK
- U2 pad 23: unconnected-(U2-I2S_LRCLK-Pad23) -> /CODEC_LRCLK
- U2 pad 24: unconnected-(U2-I2S_SCLK-Pad24) -> /CODEC_SCLK
- U2 pad 25: unconnected-(U2-I2S_DOUT-Pad25) -> /CODEC_DOUT
- U2 pad 26: unconnected-(U2-I2S_DIN-Pad26) -> /CODEC_DIN
- U2 pad 27: unconnected-(U2-CTRL_DATA-Pad27) -> /CODEC_SDA
- U2 pad 29: unconnected-(U2-CTRL_CLK-Pad29) -> /CODEC_SCL
- U2 pad 30: unconnected-(U2-VDDD-Pad30) -> +1V8
- U2 pad 31: unconnected-(U2-CTRL_ADR0_CS-Pad31) -> GND
- U2 pad 32: unconnected-(U2-CTRL_MODE-Pad32) -> GND
- U2 pad 5: unconnected-(U2-VDDA-Pad5) -> +3.3VA
- U5 pad 1: unconnected-(U5-PE2-Pad1) -> /CODEC_MCLK
- U5 pad 103: unconnected-(U5-PA11-Pad103) -> /USB_DM
- U5 pad 104: unconnected-(U5-PA12-Pad104) -> /USB_DP
- U5 pad 106: unconnected-(U5-VCAP_2-Pad106) -> /VCAP_2
- U5 pad 111: unconnected-(U5-PC10-Pad111) -> /SD_DAT2
- U5 pad 112: unconnected-(U5-PC11-Pad112) -> /SD_DAT3
- U5 pad 113: unconnected-(U5-PC12-Pad113) -> /SD_CLK
- U5 pad 116: unconnected-(U5-PD2-Pad116) -> /SD_CMD
- U5 pad 137: unconnected-(U5-PB7-Pad137) -> /SD_DETECT
- U5 pad 139: unconnected-(U5-PB8-Pad139) -> /CODEC_SCL
- U5 pad 140: unconnected-(U5-PB9-Pad140) -> /CODEC_SDA
- U5 pad 18: unconnected-(U5-PF6-Pad18) -> /ADC3_IN4
- U5 pad 19: unconnected-(U5-PF7-Pad19) -> /ADC3_IN5
- U5 pad 2: unconnected-(U5-PE3-Pad2) -> /CODEC_DOUT
- U5 pad 20: unconnected-(U5-PF8-Pad20) -> /ADC3_IN6
- U5 pad 21: unconnected-(U5-PF9-Pad21) -> /ADC3_IN7
- U5 pad 22: unconnected-(U5-PF10-Pad22) -> /ADC3_IN8
- U5 pad 27: unconnected-(U5-PC1-Pad27) -> /ADC3_IN11
- U5 pad 28: unconnected-(U5-PC2-Pad28) -> /ADC3_IN12
- U5 pad 29: unconnected-(U5-PC3-Pad29) -> /ADC3_IN13
- U5 pad 3: unconnected-(U5-PE4-Pad3) -> /CODEC_LRCLK
- U5 pad 34: unconnected-(U5-PA0-Pad34) -> /VCP_TX
- U5 pad 35: unconnected-(U5-PA1-Pad35) -> /VCP_RX
- U5 pad 36: unconnected-(U5-PA2-Pad36) -> /ADC3_IN2
- U5 pad 37: unconnected-(U5-PA3-Pad37) -> /ADC3_IN3
- U5 pad 4: unconnected-(U5-PE5-Pad4) -> /CODEC_SCLK
- U5 pad 5: unconnected-(U5-PE6-Pad5) -> /CODEC_DIN
- U5 pad 69: unconnected-(U5-PB10-Pad69) -> /PB10
- U5 pad 70: unconnected-(U5-PB11-Pad70) -> /PB11
- U5 pad 71: unconnected-(U5-VCAP_1-Pad71) -> /VCAP_1
- U5 pad 81: unconnected-(U5-PD12-Pad81) -> /PD12
- U5 pad 82: unconnected-(U5-PD13-Pad82) -> /PD13
- U5 pad 98: unconnected-(U5-PC8-Pad98) -> /SD_DAT0
- U5 pad 99: unconnected-(U5-PC9-Pad99) -> /SD_DAT1
Routing:
- net /CODEC_MCLK: track 0.00 -> 49.0 mm, vias 0 -> 2
- net /CODEC_LRCLK: track 0.00 -> 46.7 mm, vias 0 -> 2
- net +3.3VA: track 1.24 -> 46.7 mm, vias 1 -> 2
- net /SWCLK: track 0.00 -> 45.5 mm, vias 0 -> 2
- net /CODEC_SCLK: track 0.00 -> 44.5 mm, vias 0 -> 2
- net /SWDIO: track 0.00 -> 43.4 mm, vias 0 -> 2
- net /ADC3_IN3: track 0.00 -> 39.6 mm, vias 0 -> 1
- net /CODEC_DIN: track 0.00 -> 38.9 mm, vias 0 -> 2
- net /CODEC_DOUT: track 0.00 -> 38.8 mm, vias 0 -> 2
- net /SD_DAT1: track 0.00 -> 36.9 mm, vias 0 -> 2
- net /ADC3_IN4: track 0.00 -> 36.0 mm, vias 0 -> 1
- net /CODEC_SDA: track 0.00 -> 35.7 mm, vias 0 -> 2
- net /SD_DAT0: track 0.00 -> 35.6 mm
- net /SWO: track 0.00 -> 34.8 mm, vias 0 -> 2
- net /CODEC_SCL: track 0.00 -> 33.5 mm, vias 0 -> 2
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