File: hardware/dsp_som_test/dsp_som.kicad_pcb (KiCad board)
At the start: 6 copper layers, 40 x 60 mm, 61 parts, among them J1 Micro_SD_Card_Det_Hirose_DM3AT, J2 SWD, J3 DSP_SoM Connector, U1 IS42S16400J-xT, U2 SGTL5000XNLA3, U4 BU18SD2MG-MTR, U5 STM32F446ZCTx, Y1 16MHz, Y3 32kHz768

Commit message: fab
Other:
- board text removed: "JLCJLCJLCJLC"
Changed lines of the file:
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@@
 		)
 		(pad_to_mask_clearance 0)
-		(pad_to_paste_clearance_ratio -0.1)
 		(allow_soldermask_bridges_in_footprints no)
 		(pcbplotparams
@@
 			(usegerberattributes yes)
 			(usegerberadvancedattributes yes)
-			(creategerberjobfile no)
+			(creategerberjobfile yes)
 			(dashed_line_dash_ratio 12.000000)
 			(dashed_line_gap_ratio 3.000000)
@@
 			(outputformat 1)
 			(mirror no)
-			(drillshape 0)
+			(drillshape 1)
 			(scaleselection 1)
-			(outputdirectory "../gerber/")
+			(outputdirectory "")
 		)
 	)
@@
 		(layer "Edge.Cuts")
 	)
-	(gr_text "JLCJLCJLCJLC"
-		(at 109 78 0)
-		(layer "F.SilkS")
-		(effects
-			(font
-				(size 1 1)
-				(thickness 0.1)
-			)
-		)
-	)
 	(gr_text "Hole to hole 0.5mm - Center to center 0.8mm\nVia to via same net 0.254mm"
