File: hardware/carry/carry/carry.kicad_sch (KiCad schematic)
At the start: 0 parts

Commit message: routing carry board
Parts:
- added H2, H3, H4, H5: MountingHole_Pad, MountingHole:MountingHole_3.2mm_M3_Pad_Via, symbol Mechanical:MountingHole_Pad
Connections:
- new net GND: H2.1, H3.1, H4.1, H5.1
