File: hardware/carry/carry/dsp_som_slot.kicad_sch (KiCad schematic)
At the start: 2 parts, among them J6 Conn_02x22_Odd_Even

Commit message: routing carry board
Parts:
- added C26, C27, C28: 100n, Capacitor_SMD:C_0603_1608Metric, symbol Device:C_Small
- added J8: Conn_01x06, Connector_PinSocket_2.54mm:PinSocket_1x06_P2.54mm_Vertical, symbol Connector_Generic:Conn_01x06
- added R20, R21, R22, R23, R24, R25: 100k, Resistor_SMD:R_0603_1608Metric, symbol Device:R_Small
- added R26, R27: 2.2k, Resistor_SMD:R_0603_1608Metric, symbol Device:R_Small
- added SW1: RotaryEncoder_Switch, Rotary_Encoder:RotaryEncoder_Alps_EC12E-Switch_Vertical_H20mm_CircularMountingHoles, symbol Device:RotaryEncoder_Switch
Connections:
- net +3.3V: now also R20.1, R22.1, R24.1, R26.1, R27.1
- net CODEC_L_IN: now also J6.43 (Pin_43); no longer J6.41 (Pin_41)
- net CODEC_OUT_L: now also J6.39 (Pin_39); no longer J6.37 (Pin_37)
- net CODEC_OUT_R: now also J6.37 (Pin_37); no longer J6.39 (Pin_39)
- net CODEC_R_IN: now also J6.41 (Pin_41); no longer J6.43 (Pin_43)
- net GND: now also C26.1, C27.1, C28.1, J8.4 (Pin_4), SW1.C, SW1.S2
- net ADC3_IN2 renamed ENC_A
- net ENC_A: now also C27.2, R23.2
- net ADC3_IN3 renamed ENC_B
- net ENC_B: now also C28.2, R25.2
- net PB10 renamed OLED_SCL
- net OLED_SCL: now also J8.2 (Pin_2), R27.2
- net PB11 renamed OLED_SDA
- net OLED_SDA: now also J8.1 (Pin_1), R26.2
- net PD12 renamed OLED_RST
- net OLED_RST: now also J8.3 (Pin_3)
- net PD13 renamed ENC_PB
- net ENC_PB: now also C26.2, R21.2
- new net: R24.2, R25.1, SW1.B
- new net: R20.2, R21.1, SW1.S1
- new net: R22.2, R23.1, SW1.A
- new net +5V: J8.6 (Pin_6)
- no-connect marks 0 -> 1

Commit message: fab files for carry board
Parts:
- added D8: LED_Small, LED_SMD:LED_0603_1608Metric, symbol Device:LED_Small
- added R28: 1k, Resistor_SMD:R_0603_1608Metric, symbol Device:R_Small
Connections:
- net ADC3_IN13: now also D8.2 (A)
- net GND: now also R28.1
- new net: D8.1 (K), R28.2
Changed lines of the file:
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@@
 	(wire
 		(pts
-			(xy 146.05 92.71) (xy 157.48 92.71)
+			(xy 146.05 92.71) (xy 175.26 92.71)
 		)
 		(stroke
@@
 	(wire
 		(pts
+			(xy 175.26 99.06) (xy 175.26 101.6)
+		)
+		(stroke
+			(width 0)
+			(type default)
+		)
+	)
+	(wire
+		(pts
 			(xy 130.81 105.41) (xy 130.81 102.87)
 		)
@@
 	(wire
 		(pts
+			(xy 175.26 93.98) (xy 175.26 92.71)
+		)
+		(stroke
+			(width 0)
+			(type default)
+		)
+	)
+	(wire
+		(pts
 			(xy 146.05 80.01) (xy 154.94 80.01)
 		)
@@
 	)
 	(symbol
+		(lib_id "Device:LED_Small")
+		(at 175.26 96.52 90)
+		(unit 1)
+		(exclude_from_sim no)
+		(in_bom yes)
+		(on_board yes)
+		(dnp no)
+		(fields_autoplaced yes)
+		(property "Reference" "D8"
+			(at 177.8 95.1864 90)
+			(effects
+				(font
+					(size 1.27 1.27)
+				)
+				(justify right)
+			)
+		)
+		(property "Value" "LED_Small"
+			(at 177.8 97.7264 90)
+			(effects
+				(font
+					(size 1.27 1.27)
+				)
+				(justify right)
+			)
+		)
+		(property "Footprint" "LED_SMD:LED_0603_1608Metric"
+			(at 175.26 96.52 90)
+			(effects
+				(font
+					(size 1.27 1.27)
+				)
+				(hide yes)
+			)
+		)
+		(property "Datasheet" "~"
+			(at 175.26 96.52 90)
+			(effects
+				(font
+					(size 1.27 1.27)
+				)
+				(hide yes)
+			)
+		)
+		(property "Description" "Light emitting diode, small symbol"
+			(at 175.26 96.52 0)
+			(effects
+				(font
+					(size 1.27 1.27)
+				)
+				(hide yes)
+			)
+		)
+		(property "Sim.Pin" "1=K 2=A"
+			(at 175.26 96.52 0)
+			(effects
+				(font
+					(size 1.27 1.27)
+				)
+				(hide yes)
+			)
+		)
+		(pin "2"
+		)
+		(pin "1"
+		)
+		(instances
+			(project "carry"
+				(path "/d8f57854-ec5e-4c5a-8ff0-596be10a8cad/79e93208-1580-4414-b27c-df1fd4ece65b"
+					(reference "D8")
+					(unit 1)
+				)
+			)
+		)
+	)
+	(symbol
 		(lib_id "Device:C_Small")
 		(at 200.66 101.6 0)
@@
 	(symbol
 		(lib_id "Device:R_Small")
+		(at 175.26 104.14 180)
+		(unit 1)
+		(exclude_from_sim no)
+		(in_bom yes)
+		(on_board yes)
+		(dnp no)
+		(fields_autoplaced yes)
+		(property "Reference" "R28"
+			(at 177.8 102.8699 0)
+			(effects
+				(font
+					(size 1.016 1.016)
+				)
+				(justify right)
+			)
+		)
+		(property "Value" "1k"
+			(at 177.8 105.4099 0)
+			(effects
+				(font
+					(size 1.27 1.27)
+				)
+				(justify right)
+			)
+		)
+		(property "Footprint" "Resistor_SMD:R_0603_1608Metric"
+			(at 175.26 104.14 0)
+			(effects
+				(font
+					(size 1.27 1.27)
+				)
+				(hide yes)
+			)
+		)
+		(property "Datasheet" "~"
+			(at 175.26 104.14 0)
+			(effects
+				(font
+					(size 1.27 1.27)
+				)
+				(hide yes)
+			)
+		)
+		(property "Description" "Resistor, small symbol"
+			(at 175.26 104.14 0)
+			(effects
+				(font
+					(size 1.27 1.27)
+				)
+				(hide yes)
+			)
+		)
+		(pin "2"
+		)
+		(pin "1"
+		)
+		(instances
+			(project "carry"
+				(path "/d8f57854-ec5e-4c5a-8ff0-596be10a8cad/79e93208-1580-4414-b27c-df1fd4ece65b"
+					(reference "R28")
+					(unit 1)
+				)
+			)
+		)
+	)
+	(symbol
+		(lib_id "Device:R_Small")
 		(at 205.74 80.01 270)
 		(mirror x)
@@
 					(unit 1)
 				)
+			)
+		)
+	)
+	(symbol
+		(lib_id "power:GND")
+		(at 175.26 106.68 0)
+		(unit 1)
+		(exclude_from_sim no)
+		(in_bom yes)
+		(on_board yes)
+		(dnp no)
+		(fields_autoplaced yes)
+		(property "Reference" "#PWR053"
+			(at 175.26 113.03 0)
+			(effects
+				(font
+					(size 1.27 1.27)
+				)
+				(hide yes)
+			)
+		)
+		(property "Value" "GND"
+			(at 175.26 111.76 0)
+			(effects
+				(font
+					(size 1.27 1.27)
+				)
+				(hide yes)
+			)
+		)
+		(property "Footprint" ""
+			(at 175.26 106.68 0)
+			(effects
+				(font
+					(size 1.27 1.27)
+				)
+				(hide yes)
+			)
+		)
+		(property "Datasheet" ""
+			(at 175.26 106.68 0)
+			(effects
+				(font
+					(size 1.27 1.27)
+				)
+				(hide yes)
+			)
+		)
+		(property "Description" "Power symbol creates a global label with name \"GND\" , ground"
+			(at 175.26 106.68 0)
+			(effects
+				(font
+					(size 1.27 1.27)
+				)
+				(hide yes)
+			)
+		)
+		(pin "1"
+		)
+		(instances
+			(project "carry"
+				(path "/d8f57854-ec5e-4c5a-8ff0-596be10a8cad/79e93208-1580-4414-b27c-df1fd4ece65b"
+					(reference "#PWR053")
+					(unit 1)
+				)
