File: hardware/carry/carry/power_supply.kicad_sch (KiCad schematic)
At the start: 21 parts, among them J5 694106301002, J7 JST XH, U3 AZ1117CH2-5.0, U4 BU33SD5WG-TR, U5 BU33SD5WG-TR

Commit message: bom
Parts:
- D6: value BAT165A -> NSR1020MW2T1G
Changed lines of the file:
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@@
 			)
 		)
-		(property "Value" "BAT165A"
+		(property "Value" "NSR1020MW2T1G"
 			(at 83.82 34.29 0)
 			(effects
